Commit message: 完善模型

File: src/roscar_gazebo/urdf/senior_diff_gazebo.urdf (robot description, URDF)
Before this commit: robot wheeltec_robot, 8 links, 7 joints
Joints:
- joint front_wheel_joint: origin xyz=0.23 0 0.05 rpy=1.57 0 0 -> xyz=0.23 0 0.05 rpy=0 0 0
- joint left_wheel_joint: origin xyz=0 0.165 0.05 rpy=1.57 0 0 -> xyz=0 0.165 0.05 rpy=0 0 0
- joint right_wheel_joint: origin xyz=0 -0.165 0.05 rpy=1.57 0 0 -> xyz=0 -0.165 0.05 rpy=0 0 0
